File: PREAMP/HARDWARE/PREAMP/PREAMP.kicad_pcb (KiCad board)
At the start: 2 copper layers, 50 x 112 mm, 40 parts, among them J1 Input, J2 Meter Input, J3 POWER INPUT, J4 FX Input, J5 Meter Output, J6 Output, J7 BALANCED OUTPUT, J8 Power LED, U1 TL074

Commit message: PREAMP V02 and HEADPHONE AMP
Parts:
- added C11: 1uF, Capacitor_THT:C_Disc_D5.0mm_W2.5mm_P5.00mm, F.Cu at (128.0, 55.8)
- added C12: 10uF, Capacitor_THT:CP_Radial_D8.0mm_P3.80mm, F.Cu at (120.0, 64.6)
- added D5: 1N4148, Diode_THT:D_DO-35_SOD27_P7.62mm_Horizontal, F.Cu at (139.9, 72.8)
- added D6: 1N4148, Diode_THT:D_DO-35_SOD27_P7.62mm_Horizontal, F.Cu at (147.6, 75.8)
- added R12: 1M, Potentiometer_THT:Potentiometer_Piher_PT-10-V10_Vertical, F.Cu at (127.6, 64.2)
- J3: value POWER INPUT -> Conn_02x08_Odd_Even
- moved C5 11.2 mm to (120.0, 73.8), turned to 90 degrees
- moved R5 5.83 mm to (124.2, 55.8)
- moved R3 5.25 mm to (122.4, 80.2)
- moved R4 4.75 mm to (122.4, 83.8)
- moved R11 3.77 mm to (126.2, 59.8)
- moved U1 2.88 mm to (122.4, 87.9)
- moved C2 2.02 mm to (128.8, 107.2)
- moved R6 1.04 mm to (106.0, 65.2)
- moved R7 0.96 mm to (141.0, 65.0)
- moved R2 0.94 mm to (104.4, 73.0)
- moved R9 0.94 mm to (112.1, 77.0)
- moved J4 0.75 mm to (106.7, 82.2)
Connections:
- J5 pad 1: Net-(C8-Pad2) -> Net-(J5-Pad1)
Routing:
- net Net-(J5-Pad1): track 0.00 -> 71.1 mm
- net Net-(J6-Pad1): track 124.9 -> 159.9 mm
- net Earth: track 18.3 -> 50.5 mm, vias 0 -> 4
- net Net-(D5-Pad1): track 0.00 -> 24.5 mm
- net Net-(C8-Pad2): track 78.0 -> 60.5 mm, vias 2 -> 0
- net Net-(C5-Pad1): track 41.4 -> 28.2 mm
- net Net-(C4-Pad2): track 80.7 -> 92.6 mm
- net Net-(J8-Pad2): track 13.4 -> 8.57 mm
- net Net-(D1-Pad1): track 46.8 -> 42.6 mm
- net Net-(R3-Pad1): track 19.2 -> 16.5 mm
- net Net-(C1-Pad2): track 82.8 -> 80.5 mm
- net Net-(C10-Pad2): track 86.4 -> 88.4 mm
- net Net-(C4-Pad1): track 13.7 -> 15.3 mm
- net Net-(C2-Pad1): track 75.7 -> 77.2 mm
- net Net-(C8-Pad1): track 15.8 -> 14.6 mm
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- added copper zone on F.Cu, net Earth
Other:
- board text added: "Ezer Longinus Feb 2023"
- board text removed: "Ezer Longinus Jan 2023"
