File: PREAMP/HARDWARE/PREAMP/PREAMP.kicad_sch (KiCad schematic)
At the start: 1 part, among them U1 TL074

Commit message: Schematic V01
Parts:
- added C1, C2: 4.7pF, Capacitor_THT:C_Disc_D5.0mm_W2.5mm_P5.00mm, symbol Device:C_Small
- added C10, C6, C7, C8, C9: 10uF, Capacitor_THT:CP_Radial_D8.0mm_P3.80mm, symbol Device:C_Polarized_Small_US
- added C3: 100nF, Capacitor_THT:C_Disc_D5.0mm_W2.5mm_P5.00mm, symbol Device:C_Small
- added C4: 220nF, Capacitor_THT:C_Disc_D5.0mm_W2.5mm_P5.00mm, symbol Device:C_Small
- added C5: 2.2uF, Capacitor_THT:CP_Radial_D8.0mm_P3.80mm, symbol Device:C_Polarized_Small_US
- added D1, D2: LED, symbol Device:LED
- added D3, D4: 1N4001, Diode_THT:D_DO-41_SOD81_P10.16mm_Horizontal, symbol Diode:1N4001
- added J?: FX Input, Connector_Molex:Molex_SL_171971-0002_1x02_P2.54mm_Vertical, symbol Connector:Conn_01x02_Male
- added J?: Input, Connector_Molex:Molex_SL_171971-0002_1x02_P2.54mm_Vertical, symbol Connector:Conn_01x02_Male
- added J?: Meter Output, Connector_Molex:Molex_SL_171971-0002_1x02_P2.54mm_Vertical, symbol Connector:Conn_01x02_Male
- added J?: Output, Connector_Molex:Molex_SL_171971-0002_1x02_P2.54mm_Vertical, symbol Connector:Conn_01x02_Male
- added J?: BALANCED OUTPUT, symbol Connector:Conn_01x03_Male
- added J?: Meter Input, Connector_Molex:Molex_SL_171971-0002_1x02_P2.54mm_Vertical, symbol Connector:Conn_01x02_Male
- added J?: Conn_02x08_Odd_Even, Connector_IDC:IDC-Header_2x08_P2.54mm_Vertical, symbol Connector_Generic:Conn_02x08_Odd_Even
- added JP?: Jumper_2_Open, Connector_PinSocket_2.54mm:PinSocket_1x02_P2.54mm_Vertical, symbol Jumper:Jumper_2_Open
- added R1: 1k, Resistor_THT:R_Axial_DIN0207_L6.3mm_D2.5mm_P7.62mm_Horizontal, symbol Device:R_Small_US
- added R10, R9: 470k, Resistor_THT:R_Axial_DIN0207_L6.3mm_D2.5mm_P7.62mm_Horizontal, symbol Device:R_Small_US
- added R11: 1M, Resistor_THT:R_Axial_DIN0207_L6.3mm_D2.5mm_P7.62mm_Horizontal, symbol Device:R_Small_US
- added R2: 4k7, Resistor_THT:R_Axial_DIN0207_L6.3mm_D2.5mm_P7.62mm_Horizontal, symbol Device:R_Small_US
- added R3, R4: 10k, Resistor_THT:R_Axial_DIN0207_L6.3mm_D2.5mm_P7.62mm_Horizontal, symbol Device:R_Small_US
- added R6: GAIN POT, symbol Connector:Conn_01x03_Male
- added R7: MASTER, symbol Connector:Conn_01x03_Male
- added R8: 100k, Resistor_THT:R_Axial_DIN0207_L6.3mm_D2.5mm_P7.62mm_Horizontal, symbol Device:R_Small_US
- added S1: CLEAN/DIRTY, Connector_Molex:Molex_SL_171971-0002_1x02_P2.54mm_Vertical, symbol Connector:Conn_01x02_Male
Connections:
- net at U1.5 (+): now also C4.1, R8.1
- net at U1.6 (-): now also U1.7, C8.1
- net Earth: now reaches U1.10 (+)
- net Earth: now also U1.12 (+), C1.1, C10.1, C9.2, J?.1 (Pin_1), J?.1 (Pin_1), J?.2 (Pin_2), J?.2 (Pin_2), J?.2 (Pin_2), J?.2 (Pin_2), J?.3 (Pin_3), J?.4 (Pin_4), J?.5 (Pin_5), J?.6 (Pin_6), J?.7 (Pin_7), J?.8 (Pin_8), R11.2, R6.1 (Pin_1), R7.1 (Pin_1), R8.2, R9.2
- net at U1.8: now also C2.1, C6.1, R10.2, S1.1 (Pin_1)
- net at U1.9 (-): now also C2.2, D1.2 (A), D2.1 (K), R10.1, R2.2
- net at U1.13 (-): now also R3.1, R4.1
- net at U1.14: now also C7.1, R4.2
- net at U1.11 (V-): now also C10.2, D4.2 (A)
- net at U1.4 (V+): now also C9.1, D3.1 (K)
- net at U1.1: now also U1.2 (-), C5.1, R1.2
- net at U1.3 (+): now also C1.2, C3.2, R9.1
- new net: C3.1, J?.1 (Pin_1)
- new net: C5.2, R6.3 (Pin_3)
- new net: J?.2 (Pin_2), R1.1
- new net: C6.2, R7.3 (Pin_3)
- new net: C4.2, J?.1 (Pin_1), JP?.1 (A), R11.1
- new net: J?.1 (Pin_1), J?.2 (Pin_2), JP?.2 (B), R3.2, R7.2 (Pin_2)
- new net: C8.2, J?.1 (Pin_1)
- new net: R2.1, R6.2 (Pin_2)
- new net: D1.1 (K), D2.2 (A), S1.2 (Pin_2)
- new net: C7.2, J?.3 (Pin_3)
- new net +12V: D3.2 (A), J?.10 (Pin_10), J?.9 (Pin_9)
- new net +5V: J?.11 (Pin_11), J?.12 (Pin_12)
- new net -12V: D4.1 (K), J?.1 (Pin_1), J?.2 (Pin_2)
- new net CV: J?.13 (Pin_13), J?.14 (Pin_14)
- new net GATE: J?.15 (Pin_15), J?.16 (Pin_16)
Other:
- note added: "POWER INPUT"
- note added: "PREAMP"
- moved on the sheet: U1A, U1B, U1C, U1D, U1E

Commit message: Initial Board Layout
Parts:
- added H1, H2, H3, H4: MountingHole, MountingHole:MountingHole_3.2mm_M3_DIN965_Pad, symbol Mechanical:MountingHole
- C10, C9: footprint Capacitor_THT:CP_Radial_D8.0mm_P3.80mm -> Capacitor_THT:CP_Radial_D10.0mm_P3.80mm
- D1, D2: footprint (none) -> LED_THT:LED_D5.0mm
- J7: renamed from J?; footprint (none) -> Connector_Molex:Molex_SL_171971-0003_1x03_P2.54mm_Vertical
- R6, R7: footprint (none) -> Connector_Molex:Molex_SL_171971-0003_1x03_P2.54mm_Vertical
- gave numbers to parts that had none: 7

Commit message: Metronome Initial Commit
Parts:
- added J8: Power LED, Connector_Molex:Molex_SL_171971-0002_1x02_P2.54mm_Vertical, symbol Connector:Conn_01x02_Male
- added R5: 1k, Resistor_THT:R_Axial_DIN0207_L6.3mm_D2.5mm_P7.62mm_Horizontal, symbol Device:R_Small_US
Connections:
- net Earth: now also R5.1
- net at C9.1, D3.1 (K), U1.4 (V+): now also J8.1 (Pin_1)
- new net: J8.2 (Pin_2), R5.2
Changed lines of the file:
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@@
   (junction (at 67.31 50.8) (diameter 0) (color 0 0 0 0)
   )
+  (junction (at 127 144.78) (diameter 0) (color 0 0 0 0)
+  )
   (junction (at 153.035 74.295) (diameter 0) (color 0 0 0 0)
   )
@@
     (stroke (width 0) (type default) (color 0 0 0 0))
   )
+  (wire (pts (xy 137.16 147.32) (xy 137.16 149.225))
+    (stroke (width 0) (type default) (color 0 0 0 0))
+  )
   (wire (pts (xy 139.7 45.085) (xy 139.7 50.8))
     (stroke (width 0) (type default) (color 0 0 0 0))
@@
     (stroke (width 0) (type default) (color 0 0 0 0))
   )
+  (wire (pts (xy 127 144.78) (xy 139.065 144.78))
+    (stroke (width 0) (type default) (color 0 0 0 0))
+  )
   (wire (pts (xy 45.72 64.77) (xy 45.72 66.04))
     (stroke (width 0) (type default) (color 0 0 0 0))
   )
   (wire (pts (xy 85.09 153.035) (xy 83.82 153.035))
+    (stroke (width 0) (type default) (color 0 0 0 0))
+  )
+  (wire (pts (xy 139.065 147.32) (xy 137.16 147.32))
     (stroke (width 0) (type default) (color 0 0 0 0))
   )
@@
     (pin "1")
   )
+  (symbol (lib_id "power:Earth") (at 137.16 154.305 0) (unit 1)
+    (in_bom yes) (on_board yes) (fields_autoplaced)
+    (property "Reference" "#PWR026" (id 0) (at 137.16 160.655 0)
+      (effects (font (size 1.27 1.27)) hide)
+    )
+    (property "Value" "Earth" (id 1) (at 137.16 158.115 0)
+      (effects (font (size 1.27 1.27)) hide)
+    )
+    (property "Footprint" "" (id 2) (at 137.16 154.305 0)
+      (effects (font (size 1.27 1.27)) hide)
+    )
+    (property "Datasheet" "~" (id 3) (at 137.16 154.305 0)
+      (effects (font (size 1.27 1.27)) hide)
+    )
+    (pin "1")
+  )
   (symbol (lib_id "power:-12V") (at 97.79 166.37 180) (unit 1)
     (in_bom yes) (on_board yes) (fields_autoplaced)
@@
     (pin "1")
   )
+  (symbol (lib_id "Device:R_Small_US") (at 137.16 151.765 180) (unit 1)
+    (in_bom yes) (on_board yes)
+    (property "Reference" "R5" (id 0) (at 134.62 154.94 90))
+    (property "Value" "1k" (id 1) (at 134.62 149.225 90))
+    (property "Footprint" "Resistor_THT:R_Axial_DIN0207_L6.3mm_D2.5mm_P7.62mm_Horizontal" (id 2) (at 137.16 151.765 0)
+      (effects (font (size 1.27 1.27)) hide)
+    )
+    (property "Datasheet" "~" (id 3) (at 137.16 151.765 0)
+      (effects (font (size 1.27 1.27)) hide)
+    )
+    (pin "1")
+    (pin "2")
+  )
   (symbol (lib_id "power:Earth") (at 46.355 98.425 0) (unit 1)
     (in_bom yes) (on_board yes) (fields_autoplaced)
@@
     )
     (property "Datasheet" "~" (id 3) (at 129.54 78.105 0)
+      (effects (font (size 1.27 1.27)) hide)
+    )
+    (pin "1")
+    (pin "2")
+  )
+  (symbol (lib_id "Connector:Conn_01x02_Male") (at 144.145 144.78 0) (mirror y) (unit 1)
+    (in_bom yes) (on_board yes)
+    (property "Reference" "J8" (id 0) (at 141.605 138.43 0)
+      (effects (font (size 1.27 1.27)) (justify right))
+    )
+    (property "Value" "Power LED" (id 1) (at 136.525 141.605 0)
+      (effects (font (size 1.27 1.27)) (justify right))
+    )
+    (property "Footprint" "Connector_Molex:Molex_SL_171971-0002_1x02_P2.54mm_Vertical" (id 2) (at 144.145 144.78 0)
+      (effects (font (size 1.27 1.27)) hide)
+    )
+    (property "Datasheet" "~" (id 3) (at 144.145 144.78 0)
       (effects (font (size 1.27 1.27)) hide)
     )
@@
       (reference "#PWR025") (unit 1) (value "Earth") (footprint "")
     )
+    (path "/2a57ecc1-a753-4f8b-a45b-64523d80887b"
+      (reference "#PWR026") (unit 1) (value "Earth") (footprint "")
+    )
     (path "/51821289-9332-4891-85a1-3489294ba463"
       (reference "C1") (unit 1) (value "4.7pF") (footprint "Capacitor_THT:C_Disc_D5.0mm_W2.5mm_P5.00mm")
@@
       (reference "J7") (unit 1) (value "BALANCED OUTPUT") (footprint "Connector_Molex:Molex_SL_171971-0003_1x03_P2.54mm_Vertical")
     )
+    (path "/e2d7c3d4-fc4f-4efe-9699-418b43c94919"
+      (reference "J8") (unit 1) (value "Power LED") (footprint "Connector_Molex:Molex_SL_171971-0002_1x02_P2.54mm_Vertical")
+    )
     (path "/72ea267e-47e6-4c1d-96fa-150ba46275c8"
       (reference "JP1") (unit 1) (value "Jumper_2_Open") (footprint "Connector_PinSocket_2.54mm:PinSocket_1x02_P2.54mm_Vertical")
@@
       (reference "R4") (unit 1) (value "10k") (footprint "Resistor_THT:R_Axial_DIN0207_L6.3mm_D2.5mm_P7.62mm_Horizontal")
     )
+    (path "/8c9fc5ef-9f2f-4196-a1d7-af8b8604d5b6"
+      (reference "R5") (unit 1) (value "1k") (footprint "Resistor_THT:R_Axial_DIN0207_L6.3mm_D2.5mm_P7.62mm_Horizontal")
+    )
     (path "/854155d4-d606-4772-8770-9158b1cdf63e"

Commit message: Production Files Fixed
Parts:
- added C11: 1uF, Capacitor_THT:C_Disc_D5.0mm_W2.5mm_P5.00mm, symbol Device:C_Small
- added C12: 10uF, Capacitor_THT:CP_Radial_D8.0mm_P3.80mm, symbol Device:C_Polarized_Small_US
- added D5, D6: 1N4148, Diode_THT:D_DO-35_SOD27_P7.62mm_Horizontal, symbol Diode:1N4148
- added R12: 1M, Potentiometer_THT:Potentiometer_Piher_PT-10-V10_Vertical, symbol Device:R_Potentiometer_US
Connections:
- net Earth: now also C11.2, C12.2, D5.2 (A)
- net at J5.1 (Pin_1): now also C11.1, C12.1, D6.1 (K); no longer C8.2
- new net: D5.1 (K), D6.2 (A), R12.2, R12.3
- new net: C8.2, R12.1
Other:
- moved on the sheet: J5
