File: METRONOME/Hardware/METRONOME/METRONOME.kicad_pcb (KiCad board)
At the start: 2 copper layers, 50 x 112 mm, 40 parts, among them J1 Input, J2 Meter Input, J3 POWER INPUT, J4 FX Input, J5 Meter Output, J6 Output, J7 BALANCED OUTPUT, J8 Power LED, U1 TL074

Commit message: Initial Metronome Layout Commit
Parts:
- removed C5: 2.2uF, Capacitor_THT:CP_Radial_D8.0mm_P3.80mm
- removed C6, C7, C8: 10uF, Capacitor_THT:CP_Radial_D8.0mm_P3.80mm
- removed D1, D2: LED, LED_THT:LED_D5.0mm
- removed J4: FX Input, Connector_Molex:Molex_SL_171971-0002_1x02_P2.54mm_Vertical
- removed J5: Meter Output, Connector_Molex:Molex_SL_171971-0002_1x02_P2.54mm_Vertical
- removed J7: BALANCED OUTPUT, Connector_Molex:Molex_SL_171971-0003_1x03_P2.54mm_Vertical
- removed JP1: Jumper_2_Open, Connector_PinSocket_2.54mm:PinSocket_1x02_P2.54mm_Vertical
- removed R10, R9: 470k, Resistor_THT:R_Axial_DIN0207_L6.3mm_D2.5mm_P7.62mm_Horizontal
- removed R11: 1M, Resistor_THT:R_Axial_DIN0207_L6.3mm_D2.5mm_P7.62mm_Horizontal
- removed R8: 100k, Resistor_THT:R_Axial_DIN0207_L6.3mm_D2.5mm_P7.62mm_Horizontal
- added -12V: TestPoint, Connector_Pin:Pin_D1.2mm_L10.2mm_W2.9mm_FlatFork, F.Cu at (136.5, 125.0)
- C1, C2: value 4.7pF -> 2.2uF; footprint Capacitor_THT:C_Disc_D5.0mm_W2.5mm_P5.00mm -> Capacitor_THT:CP_Radial_D8.0mm_P3.80mm
- C3: value 100nF -> 100uF; footprint Capacitor_THT:C_Disc_D5.0mm_W2.5mm_P5.00mm -> Capacitor_THT:CP_Radial_D10.0mm_P3.80mm
- C4: value 220nF -> 100uF; footprint Capacitor_THT:C_Disc_D5.0mm_W2.5mm_P5.00mm -> Capacitor_THT:CP_Radial_D10.0mm_P3.80mm
- J1: value Input -> Output
- J2: value Meter Input -> Tempo LED
- J6: value Output -> SPEAKER
- R1: value 1k -> 1k5
- R2: value 4k7 -> 47k
- R3: value 10k -> TEMPO - 1M; footprint Resistor_THT:R_Axial_DIN0207_L6.3mm_D2.5mm_P7.62mm_Horizontal -> Connector_Molex:Molex_SL_171971-0003_1x03_P2.54mm_Vertical
- R6: value GAIN POT -> 1k; footprint Connector_Molex:Molex_SL_171971-0003_1x03_P2.54mm_Vertical -> Resistor_THT:R_Axial_DIN0207_L6.3mm_D2.5mm_P7.62mm_Horizontal
- R7: value MASTER -> 1k; footprint Connector_Molex:Molex_SL_171971-0003_1x03_P2.54mm_Vertical -> Resistor_THT:R_Axial_DIN0207_L6.3mm_D2.5mm_P7.62mm_Horizontal
- S1: value CLEAN/DIRTY -> SPKR_SW
- U1: value TL074 -> LM555xN; footprint Package_DIP:DIP-14_W7.62mm_LongPads -> Package_DIP:DIP-8_W7.62mm
- moved S1 64.6 mm to (125.2, 116.5)
- moved R6 39.5 mm to (111.6, 104.5), turned to 180 degrees
- moved C3 38.1 mm to (128.3, 79.8), turned to 180 degrees
- moved R2 33.3 mm to (136.9, 83.5)
- moved R4 31.9 mm to (111.6, 109.0), turned to 180 degrees
- moved R5 29.8 mm to (104.4, 70.5), turned to 0 degrees
- moved R3 21.9 mm to (139.5, 61.2)
- moved R1 20.6 mm to (122.9, 100.5)
- moved C1 18.9 mm to (138.7, 92.2), turned to 0 degrees
- moved R7 18.2 mm to (122.7, 70.5)
- moved J2 15.1 mm to (125.2, 61.2)
- moved C2 9.78 mm to (138.7, 104.0), turned to 0 degrees
- moved J8 9.55 mm to (107.0, 61.2)
- moved C4 6.40 mm to (108.0, 92.2), turned to -90 degrees
- moved U1 3.71 mm to (122.7, 88.7)
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Connections:
- C1 pad 1: Earth -> Net-(C1-Pad1)
- C2 pad 1: Net-(C2-Pad1) -> Earth
- C2 pad 2: Net-(C2-Pad2) -> Net-(C1-Pad2)
- C3 pad 1: Net-(C3-Pad1) -> VCC
- C3 pad 2: Net-(C1-Pad2) -> Earth
- C9 pad 1: Net-(C9-Pad1) -> VCC
- D3 pad 1: Net-(C9-Pad1) -> VCC
- J1 pad 1: Net-(C3-Pad1) -> Net-(J1-Pad1)
- J2 pad 1: Net-(C4-Pad2) -> VCC
- J2 pad 2: Earth -> Net-(J2-Pad2)
- J6 pad 1: Net-(R3-Pad2) -> Net-(J6-Pad1)
- J8 pad 1: Net-(C9-Pad1) -> VCC
- R1 pad 1: Net-(R1-Pad1) -> Net-(C1-Pad1)
- R1 pad 2: Net-(C5-Pad1) -> Net-(R1-Pad2)
- R2 pad 1: Net-(R2-Pad1) -> VCC
- R2 pad 2: Net-(C2-Pad2) -> Net-(R2-Pad2)
- R3 pad 1: Net-(R3-Pad1) -> Net-(R1-Pad2)
- R3 pad 2: Net-(R3-Pad2) -> Net-(R1-Pad2)
- R4 pad 1: Net-(R3-Pad1) -> Net-(C4-Pad2)
- R4 pad 2: Net-(C7-Pad1) -> Net-(J1-Pad1)
- R6 pad 2: Net-(R2-Pad1) -> Net-(J1-Pad1)
- R7 pad 1: Earth -> Net-(C4-Pad1)
- R7 pad 2: Net-(R3-Pad2) -> Net-(J2-Pad2)
- S1 pad 1: Net-(C2-Pad1) -> Net-(C4-Pad2)
- S1 pad 2: Net-(D1-Pad1) -> Net-(J6-Pad1)
- U1 pad 1: Net-(C5-Pad1) -> Earth
- U1 pad 2: Net-(C5-Pad1) -> Net-(C1-Pad1)
- U1 pad 3: Net-(C1-Pad2) -> Net-(C4-Pad1)
- U1 pad 4: Net-(C9-Pad1) -> VCC
- U1 pad 5: Net-(C4-Pad1) -> unconnected-(U1-Pad5)
- U1 pad 6: Net-(C8-Pad1) -> Net-(C1-Pad1)
- U1 pad 7: Net-(C8-Pad1) -> Net-(R1-Pad2)
- U1 pad 8: Net-(C2-Pad1) -> VCC
Routing:
- net VCC: track 0.00 -> 134.3 mm
- net Net-(C9-Pad1): track 130.5 -> 0.00 mm
- net Net-(R3-Pad2): track 124.9 -> 0.00 mm, vias 2 -> 0
- net Net-(C8-Pad2): track 78.0 -> 0.00 mm, vias 2 -> 0
- net Net-(C2-Pad2): track 76.3 -> 0.00 mm, vias 4 -> 0
- net Net-(C2-Pad1): track 75.7 -> 0.00 mm, vias 2 -> 0
- net Net-(C1-Pad2): track 82.8 -> 11.8 mm
- net Net-(C10-Pad2): track 86.4 -> 25.2 mm
- net Net-(R1-Pad2): track 0.00 -> 52.5 mm
- net Net-(C1-Pad1): track 0.00 -> 48.2 mm, vias 0 -> 4
- net Net-(D1-Pad1): track 46.8 -> 0.00 mm, vias 2 -> 0
- net Net-(C4-Pad2): track 80.7 -> 35.1 mm, vias 0 -> 2
- net Net-(C7-Pad1): track 43.4 -> 0.00 mm, vias 2 -> 0
- net Net-(C6-Pad2): track 43.0 -> 0.00 mm
- net Net-(C5-Pad1): track 41.4 -> 0.00 mm
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Other:
- board text added: "EPFM - METRONOME"
- board text removed: "EPFM - PREAMP"
