File: MINI_AMP/Hardware/MINI_AMP/MINI_AMP.kicad_sch (KiCad schematic)
At the start: 30 parts, among them J1 INPUT 1, J2 INPUT 2, J3 Conn_02x08_Odd_Even, J4 OUTPUT 2, J6 OUTPUT 1, J8 Power LED, U1 LM380N

Commit message: PREAMP V02 and HEADPHONE AMP
Parts:
- removed C2: 10nF, Capacitor_THT:C_Disc_D5.0mm_W2.5mm_P5.00mm, symbol Device:C_Small
- removed C5: 10uF, Capacitor_THT:CP_Radial_D8.0mm_P3.80mm, symbol Device:C_Polarized_Small_US
- removed C6: 220uF, Capacitor_THT:CP_Radial_D14.0mm_P5.00mm, symbol Device:C_Polarized_Small_US
- removed D1, D2: 1N4001, Diode_THT:D_DO-41_SOD81_P10.16mm_Horizontal, symbol Diode:1N4001
- removed J4: OUTPUT 2, Connector_Molex:Molex_SL_171971-0002_1x02_P2.54mm_Vertical, symbol Connector:Conn_01x02_Male
- removed R3: VOL 250k, Connector_Molex:Molex_SL_171971-0003_1x03_P2.54mm_Vertical, symbol Connector:Conn_01x03_Male
- removed R4: 100k, Resistor_THT:R_Axial_DIN0207_L6.3mm_D2.5mm_P7.62mm_Horizontal, symbol Device:R_Small_US
- removed R5: 470k, Resistor_THT:R_Axial_DIN0207_L6.3mm_D2.5mm_P7.62mm_Horizontal, symbol Device:R_Small_US
- removed U1: LM380N, Package_DIP:DIP-14_W7.62mm, symbol Amplifier_Audio:LM380N
- added C2: 10uF, Capacitor_THT:CP_Radial_D10.0mm_P3.80mm, symbol Device:C_Polarized_Small_US
- added C5: 220nF, Capacitor_THT:C_Disc_D5.0mm_W2.5mm_P5.00mm, symbol Device:C_Small
- added C6: 100nF, Capacitor_THT:C_Disc_D5.0mm_W2.5mm_P5.00mm, symbol Device:C_Small
- added C7: 470uF, Capacitor_THT:CP_Radial_D14.0mm_P5.00mm, symbol Device:C_Polarized_Small_US
- added J10: HEADPHONE_B, Connector_Molex:Molex_SL_171971-0003_1x03_P2.54mm_Vertical, symbol Connector:Conn_01x03_Male
- added J4: Barrel_Jack_Switch, Connector_BarrelJack:BarrelJack_GCT_DCJ200-10-A_Horizontal, symbol Connector:Barrel_Jack_Switch
- added J5: PWR_SW_A, Connector_Molex:Molex_SL_171971-0002_1x02_P2.54mm_Vertical, symbol Connector:Conn_01x02_Male
- added J7: PWR_SW_B, Connector_Molex:Molex_SL_171971-0002_1x02_P2.54mm_Vertical, symbol Connector:Conn_01x02_Male
- added J9: HEADPHONE_A, Connector_Molex:Molex_SL_171971-0003_1x03_P2.54mm_Vertical, symbol Connector:Conn_01x03_Male
- added R10, R9: IN_VOL_1M, Connector_Molex:Molex_SL_171971-0003_1x03_P2.54mm_Vertical, symbol Connector:Conn_01x03_Male
- added R3: 33, Resistor_THT:R_Axial_DIN0207_L6.3mm_D2.5mm_P7.62mm_Horizontal, symbol Device:R_Small_US
- added R7: 100k, Resistor_THT:R_Axial_DIN0207_L6.3mm_D2.5mm_P7.62mm_Horizontal, symbol Device:R_Small_US
- added R8: 470k, Resistor_THT:R_Axial_DIN0207_L6.3mm_D2.5mm_P7.62mm_Horizontal, symbol Device:R_Small_US
- added S1: OUT_SW, Connector_Molex:Molex_SL_171971-0003_1x03_P2.54mm_Vertical, symbol Connector:Conn_01x03_Male
- added U1: LM384, Package_DIP:DIP-14_W7.62mm, symbol Amplifier_Audio:LM384
- C1: value 100pF -> 22pF
- C4: value 100nF -> 220nF
- J1: value INPUT 1 -> INPUT A
- J2: value INPUT 2 -> INPUT B
- J6: value OUTPUT 1 -> SPEAKER
- R1: value 3.3 -> 2.7
- R2: value 10 -> 33
- R5: renamed from R7; value 3k3 -> 1k
- R6: value 470k -> 100k
Connections:
- net +12V: now also J4.1, J5.1 (Pin_1); no longer D3.2 (A)
- net -12V: now also J4.2, J7.2 (Pin_2); no longer D4.1 (K), J3.1 (Pin_1), J3.2 (Pin_2)
- net Earth: now also D4.2 (A), C2.2, C6.1, J10.3 (Pin_3), J9.3 (Pin_3), R10.1 (Pin_1), R8.1, R9.1 (Pin_1), U1.10 (GND), U1.11 (GND), U1.12 (GND), U1.2 (+), U1.3 (GND), U1.4 (GND), U1.5 (GND), U1.7 (GND); no longer C4.2
- net at R1.2: now also C7.1, U1.8; no longer C3.2
- net at J6.1 (Pin_1): now also S1.3 (Pin_3)
- net +24V: now reaches D3.1 (K)
- net +24V: now also C3.2, C9.1, J8.1 (Pin_1), U1.14 (VS)
- net at C1.2: now also C4.1, C5.1, R8.2, U1.6 (-); no longer R6.2
- net at R1.1: now also C6.2
- net at R2.1: now also J10.1 (Pin_1), J10.2 (Pin_2)
- net at J1.1 (Pin_1): now also R9.3 (Pin_3)
- net at R2.2: now also R3.2, S1.1 (Pin_1)
- net at J2.1 (Pin_1): now also R10.3 (Pin_3); no longer R6.1
- removed net +VDC: C4.1, C9.1, J8.1 (Pin_1)
- new net: C5.2, R7.2
- new net: C7.2, S1.2 (Pin_2)
- new net: C2.1, U1.1 (BYPASS)
- new net: R10.2 (Pin_2), R7.1
- new net: D4.1 (K), J7.1 (Pin_1)
- new net: C4.2, R6.2
- new net: D3.2 (A), J5.2 (Pin_2)
- new net: R6.1, R9.2 (Pin_2)
- new net: J3.1 (Pin_1), J3.2 (Pin_2), J4.3
- new net: J9.1 (Pin_1), J9.2 (Pin_2), R3.1
Other:
- note added: "MINI AMP"
- note removed: "HEADPHONE AMP"
- moved on the sheet: C1, C10, C3, C4, C9, J1, J2, J6
