File: MINI_AMP/Hardware/MINI_AMP/MINI_AMP.kicad_pcb (KiCad board)
At the start: 2 copper layers, 50 x 112 mm, 36 parts, among them J1 INPUT A, J10 HEADPHONE_B, J2 INPUT B, J3 Conn_02x08_Odd_Even, J4 Barrel_Jack_Switch, J5 PWR_SW_A, J6 SPEAKER, J7 PWR_SW_B, J8 Power LED, J9 HEADPHONE_A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

Commit message: Metronome CAD files
Parts:
- moved J4 0.82 mm to (135.6, 132.3)
Routing:
- net Net-(J3-Pad2): track 18.1 -> 18.9 mm
- added copper zone on F.Cu, net Earth

Commit message: Ultra Fuzz and PTC files
Changed lines of the file:
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@@
     (fp_line (start -2.37 -0.24) (end -2.37 1.79) (layer "F.Fab") (width 0.1))
     (fp_line (start 7.45 1.79) (end 7.45 -0.24) (layer "F.Fab") (width 0.1))
-    (pad "1" thru_hole roundrect (at 0 0 270) (size 1.74 1.74) (drill 1.09) (layers *.Cu *.Mask) (roundrect_rratio 0.143678)
+    (pad "1" thru_hole roundrect (at 0 0 270) (size 1.74 1.74) (drill 1.09) (layers *.Cu *.Mask) (roundrect_rratio 0.1436781609)
       (net 22 "Net-(J9-Pad1)") (pinfunction "Pin_1") (pintype "passive"))
     (pad "2" thru_hole circle (at 2.54 0 270) (size 1.74 1.74) (drill 1.09) (layers *.Cu *.Mask)
@@
     (fp_line (start -2.37 -0.24) (end -2.37 1.79) (layer "F.Fab") (width 0.1))
     (fp_line (start -1.27 2.55) (end -1.27 4.05) (layer "F.Fab") (width 0.1))
-    (pad "1" thru_hole roundrect (at 0 0 270) (size 1.74 1.74) (drill 1.09) (layers *.Cu *.Mask) (roundrect_rratio 0.143678)
+    (pad "1" thru_hole roundrect (at 0 0 270) (size 1.74 1.74) (drill 1.09) (layers *.Cu *.Mask) (roundrect_rratio 0.1436781609)
       (net 1 "Earth") (pinfunction "Pin_1") (pintype "passive"))
     (pad "2" thru_hole circle (at 2.54 0 270) (size 1.74 1.74) (drill 1.09) (layers *.Cu *.Mask)
@@
     (fp_line (start -2.5 -0.24) (end -2.37 -0.24) (layer "F.Fab") (width 0.1))
     (fp_line (start 6.35 4.05) (end 6.35 2.55) (layer "F.Fab") (width 0.1))
-    (pad "1" thru_hole roundrect (at 0 0 270) (size 1.74 1.74) (drill 1.09) (layers *.Cu *.Mask) (roundrect_rratio 0.143678)
+    (pad "1" thru_hole roundrect (at 0 0 270) (size 1.74 1.74) (drill 1.09) (layers *.Cu *.Mask) (roundrect_rratio 0.1436781609)
       (net 23 "Net-(J10-Pad1)") (pinfunction "Pin_1") (pintype "passive"))
     (pad "2" thru_hole circle (at 2.54 0 270) (size 1.74 1.74) (drill 1.09) (layers *.Cu *.Mask)
@@
     (fp_line (start 4.96 -0.24) (end 4.96 -2.55) (layer "F.Fab") (width 0.1))
     (fp_line (start 4.7 4.05) (end 4.7 2.55) (layer "F.Fab") (width 0.1))
-    (pad "1" thru_hole roundrect (at 0 0 270) (size 1.74 1.74) (drill 1.09) (layers *.Cu *.Mask) (roundrect_rratio 0.143678)
+    (pad "1" thru_hole roundrect (at 0 0 270) (size 1.74 1.74) (drill 1.09) (layers *.Cu *.Mask) (roundrect_rratio 0.1436781609)
       (net 9 "Net-(D4-Pad1)") (pinfunction "Pin_1") (pintype "passive"))
     (pad "2" thru_hole circle (at 2.54 0 270) (size 1.74 1.74) (drill 1.09) (layers *.Cu *.Mask)
@@
     (fp_line (start -2.42 -2.55) (end -2.42 -0.24) (layer "F.Fab") (width 0.1))
     (fp_line (start -2.16 4.05) (end 4.7 4.05) (layer "F.Fab") (width 0.1))
-    (pad "1" thru_hole roundrect (at 0 0 270) (size 1.74 1.74) (drill 1.09) (layers *.Cu *.Mask) (roundrect_rratio 0.143678)
+    (pad "1" thru_hole roundrect (at 0 0 270) (size 1.74 1.74) (drill 1.09) (layers *.Cu *.Mask) (roundrect_rratio 0.1436781609)
       (net 14 "Net-(J2-Pad1)") (pinfunction "Pin_1") (pintype "passive"))
     (pad "2" thru_hole circle (at 2.54 0 270) (size 1.74 1.74) (drill 1.09) (layers *.Cu *.Mask)
@@
     (fp_line (start -2.29 1.79) (end -2.42 1.79) (layer "F.Fab") (width 0.1))
     (fp_line (start 4.83 -0.24) (end 4.96 -0.24) (layer "F.Fab") (width 0.1))
-    (pad "1" thru_hole roundrect (at 0 0 270) (size 1.74 1.74) (drill 1.09) (layers *.Cu *.Mask) (roundrect_rratio 0.143678)
+    (pad "1" thru_hole roundrect (at 0 0 270) (size 1.74 1.74) (drill 1.09) (layers *.Cu *.Mask) (roundrect_rratio 0.1436781609)
       (net 17 "+12V") (pinfunction "Pin_1") (pintype "passive"))
     (pad "2" thru_hole circle (at 2.54 0 270) (size 1.74 1.74) (drill 1.09) (layers *.Cu *.Mask)
@@
     (fp_line (start 4.96 -0.24) (end 4.96 -2.55) (layer "F.Fab") (width 0.1))
     (fp_line (start 4.96 -2.55) (end -2.42 -2.55) (layer "F.Fab") (width 0.1))
-    (pad "1" thru_hole roundrect (at 0 0 90) (size 1.74 1.74) (drill 1.09) (layers *.Cu *.Mask) (roundrect_rratio 0.143678)
+    (pad "1" thru_hole roundrect (at 0 0 90) (size 1.74 1.74) (drill 1.09) (layers *.Cu *.Mask) (roundrect_rratio 0.1436781609)
       (net 16 "Net-(J6-Pad1)") (pinfunction "Pin_1") (pintype "passive"))
     (pad "2" thru_hole circle (at 2.54 0 90) (size 1.74 1.74) (drill 1.09) (layers *.Cu *.Mask)
@@
     (fp_line (start 0 -1.842893) (end -0.5 -2.55) (layer "F.Fab") (width 0.1))
     (fp_line (start 4.83 -0.24) (end 4.96 -0.24) (layer "F.Fab") (width 0.1))
-    (pad "1" thru_hole roundrect (at 0 0 90) (size 1.74 1.74) (drill 1.09) (layers *.Cu *.Mask) (roundrect_rratio 0.143678)
+    (pad "1" thru_hole roundrect (at 0 0 90) (size 1.74 1.74) (drill 1.09) (layers *.Cu *.Mask) (roundrect_rratio 0.1436781609)
       (net 2 "+24V") (pinfunction "Pin_1") (pintype "passive"))
     (pad "2" thru_hole circle (at 2.54 0 90) (size 1.74 1.74) (drill 1.09) (layers *.Cu *.Mask)
@@
     (fp_line (start -2.5 2.55) (end 7.58 2.55) (layer "F.Fab") (width 0.1))
     (fp_line (start 7.58 2.55) (end 7.58 1.79) (layer "F.Fab") (width 0.1))
-    (pad "1" thru_hole roundrect (at 0 0 270) (size 1.74 1.74) (drill 1.09) (layers *.Cu *.Mask) (roundrect_rratio 0.143678)
+    (pad "1" thru_hole roundrect (at 0 0 270) (size 1.74 1.74) (drill 1.09) (layers *.Cu *.Mask) (roundrect_rratio 0.1436781609)
       (net 1 "Earth") (pinfunction "Pin_1") (pintype "passive"))
     (pad "2" thru_hole circle (at 2.54 0 270) (size 1.74 1.74) (drill 1.09) (layers *.Cu *.Mask)
@@
     (fp_line (start -2.5 -0.24) (end -2.37 -0.24) (layer "F.Fab") (width 0.1))
     (fp_line (start -1.27 4.05) (end 6.35 4.05) (layer "F.Fab") (width 0.1))
-    (pad "1" thru_hole roundrect (at 0 0 270) (size 1.74 1.74) (drill 1.09) (layers *.Cu *.Mask) (roundrect_rratio 0.143678)
+    (pad "1" thru_hole roundrect (at 0 0 270) (size 1.74 1.74) (drill 1.09) (layers *.Cu *.Mask) (roundrect_rratio 0.1436781609)
       (net 24 "Net-(R2-Pad2)") (pinfunction "Pin_1") (pintype "passive"))
     (pad "2" thru_hole circle (at 2.54 0 270) (size 1.74 1.74) (drill 1.09) (layers *.Cu *.Mask)
@@
     (fp_line (start -2.42 -2.55) (end -2.42 -0.24) (layer "F.Fab") (width 0.1))
     (fp_line (start 0.5 -2.55) (end 0 -1.842893) (layer "F.Fab") (width 0.1))
-    (pad "1" thru_hole roundrect (at 0 0 270) (size 1.74 1.74) (drill 1.09) (layers *.Cu *.Mask) (roundrect_rratio 0.143678)
+    (pad "1" thru_hole roundrect (at 0 0 270) (size 1.74 1.74) (drill 1.09) (layers *.Cu *.Mask) (roundrect_rratio 0.1436781609)
       (net 13 "Net-(R9-Pad3)") (pinfunction "Pin_1") (pintype "passive"))
     (pad "2" thru_hole circle (at 2.54 0 270) (size 1.74 1.74) (drill 1.09) (layers *.Cu *.Mask)
