File: HEADPHONE_AMP/Hardware/HEADPHONE_AMP/HEADPHONE_AMP.kicad_pcb (KiCad board)
At the start: 2 copper layers, 50 x 112 mm, 28 parts, among them J1 INPUT 1, J2 INPUT 2, J3 Conn_02x08_Odd_Even, J4 OUTPUT 2, J6 OUTPUT 1, J8 Power LED, U1 LM380N

Commit message: PREAMP V02 and HEADPHONE AMP
Parts:
- added D1: 1N4001, Diode_THT:D_DO-41_SOD81_P10.16mm_Horizontal, F.Cu at (112.9, 132.2)
- added D2: 1N4001, Diode_THT:D_DO-41_SOD81_P10.16mm_Horizontal, F.Cu at (129.2, 132.2)
- C6: footprint Capacitor_THT:CP_Radial_D8.0mm_P3.80mm -> Capacitor_THT:CP_Radial_D14.0mm_P5.00mm
- R7: value 1k -> 3k3
- moved D4 10.2 mm to (129.2, 136.0), turned to 0 degrees
- moved C9 6.69 mm to (109.5, 125.2), turned to 180 degrees
- moved C10 2.82 mm to (146.0, 125.8), turned to 180 degrees
- moved C4 1.75 mm to (129.2, 121.8)
- moved C2 1.25 mm to (129.2, 118.0)
- moved C5 1.12 mm to (132.9, 121.0)
Connections:
- C10 pad 1: Earth -> Net-(J3-Pad4)
- C10 pad 2: -VDC -> Earth
- C9 pad 2: Earth -> Net-(J3-Pad4)
- D3 pad 1: +VDC -> Net-(D3-Pad1)
- D4 pad 2: -VDC -> Net-(D4-Pad2)
- J3 pad 3: Earth -> Net-(J3-Pad4)
- J3 pad 4: Earth -> Net-(J3-Pad4)
- J3 pad 5: Earth -> Net-(J3-Pad4)
- J3 pad 6: Earth -> Net-(J3-Pad4)
- J3 pad 7: Earth -> Net-(J3-Pad4)
- J3 pad 8: Earth -> Net-(J3-Pad4)
Routing:
- net Net-(J3-Pad4): track 0.00 -> 91.7 mm
- net -VDC: track 18.7 -> 0.00 mm
- net Net-(D4-Pad2): track 0.00 -> 11.7 mm
- net Net-(D3-Pad1): track 0.00 -> 11.7 mm
- net +VDC: track 155.3 -> 145.5 mm
- net Earth: track 38.1 -> 45.8 mm
- net Net-(C2-Pad1): track 10.0 -> 6.64 mm
- net Net-(C5-Pad1): track 8.58 -> 7.81 mm
- net -12V: track 12.6 -> 13.2 mm
Other:
- board text added: "Ezer Longinus Feb 2023"
- board text removed: "Ezer Longinus Jan 2023"

Commit message: Metronome CAD files
Routing:
- net +VDC: track 145.5 -> 155.1 mm
- net Net-(C2-Pad1): track 6.64 -> 8.59 mm
- added copper zone on F.Cu, net Earth
Changed lines of the file:
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@@
     (property "Sheetname" "")
     (attr through_hole)
-    (fp_text reference "D1" (at -2.42 -1) (layer "F.SilkS")
+    (fp_text reference "D1" (at -2.43 -1.0082) (layer "F.SilkS")
       (effects (font (size 1 1) (thickness 0.15)))
     )
@@
       (effects (font (size 1 1) (thickness 0.15)))
     )
-    (fp_text user "${REFERENCE}" (at -2.42 -1) (layer "F.SilkS")
-      (effects (font (size 1 1) (thickness 0.15)))
-    )
     (fp_text user "K" (at 0 -2.1) (layer "F.Fab")
+      (effects (font (size 1 1) (thickness 0.15)))
+    )
+    (fp_text user "${REFERENCE}" (at -2.42 -1) (layer "F.Fab")
       (effects (font (size 1 1) (thickness 0.15)))
     )
@@
       (effects (font (size 1 1) (thickness 0.15)))
     )
-    (fp_text value " INPUT 1" (at 1.27 5.25) (layer "F.SilkS")
+    (fp_text value " INPUT 1" (at 1.3166 5.196) (layer "F.SilkS")
       (effects (font (size 1 1) (thickness 0.15)))
     )
@@
   (segment (start 114 87.5) (end 115 87.5) (width 1) (layer "B.Cu") (net 2))
   (segment (start 102.5 90.75) (end 102.5 101.25) (width 1) (layer "B.Cu") (net 2))
+  (segment (start 129.25 118) (end 128.795 118) (width 1) (layer "B.Cu") (net 3))
   (segment (start 130.55 111.835) (end 129.165 111.835) (width 1) (layer "B.Cu") (net 3))
-  (segment (start 127.75 113.25) (end 127.75 116.5) (width 1) (layer "B.Cu") (net 3))
-  (segment (start 129.165 111.835) (end 127.75 113.25) (width 1) (layer "B.Cu") (net 3))
+  (segment (start 128.27 117.475) (end 128.27 112.73) (width 1) (layer "B.Cu") (net 3))
+  (segment (start 128.27 112.73) (end 128.4375 112.5625) (width 1) (layer "B.Cu") (net 3))
+  (segment (start 129.165 111.835) (end 128.4375 112.5625) (width 1) (layer "B.Cu") (net 3))
+  (segment (start 128.795 118) (end 128.27 117.475) (width 1) (layer "B.Cu") (net 3))
   (segment (start 130.56 94.5) (end 130.56 91.06) (width 1) (layer "B.Cu") (net 4))
   (segment (start 130.56 91.06) (end 129.25 89.75) (width 1) (layer "B.Cu") (net 4))
@@
   (segment (start 143.75 54.25) (end 149 59.5) (width 1) (layer "B.Cu") (net 5))
   (segment (start 112.92 132.08) (end 114.75 130.25) (width 1) (layer "B.Cu") (net 5))
+  (segment (start 126.365 120.65) (end 127.465 121.75) (width 1) (layer "B.Cu") (net 5))
+  (segment (start 122.93 114.375) (end 124.535 114.375) (width 1) (layer "B.Cu") (net 5))
+  (segment (start 124.535 114.375) (end 126.365 116.205) (width 1) (layer "B.Cu") (net 5))
   (segment (start 114.75 130.25) (end 126 130.25) (width 1) (layer "B.Cu") (net 5))
   (segment (start 112.92 132.25) (end 112.92 132.08) (width 1) (layer "B.Cu") (net 5))
   (segment (start 129.25 127) (end 129.25 125.5) (width 1) (layer "B.Cu") (net 5))
-  (segment (start 124.125 114.375) (end 122.93 114.375) (width 1) (layer "B.Cu") (net 5))
   (segment (start 139.75 122.25) (end 136.5 125.5) (width 1) (layer "B.Cu") (net 5))
   (segment (start 109.517677 129.767677) (end 109.517677 125.25) (width 1) (layer "B.Cu") (net 5))
-  (segment (start 126.25 116.5) (end 124.125 114.375) (width 1) (layer "B.Cu") (net 5))
+  (segment (start 129.25 125.5) (end 129.25 121.75) (width 1) (layer "B.Cu") (net 5))
   (segment (start 149 117) (end 143.75 122.25) (width 1) (layer "B.Cu") (net 5))
   (segment (start 149 59.5) (end 149 117) (width 1) (layer "B.Cu") (net 5))
@@
   (segment (start 136.5 125.5) (end 129.25 125.5) (width 1) (layer "B.Cu") (net 5))
   (segment (start 127.5 54.25) (end 143.75 54.25) (width 1) (layer "B.Cu") (net 5))
-  (segment (start 129.25 125.5) (end 129.25 123.5) (width 1) (layer "B.Cu") (net 5))
   (segment (start 112.92 132.25) (end 112 132.25) (width 1) (layer "B.Cu") (net 5))
   (segment (start 125.46 59.25) (end 125.46 56.29) (width 1) (layer "B.Cu") (net 5))
+  (segment (start 127.465 121.75) (end 129.25 121.75) (width 1) (layer "B.Cu") (net 5))
   (segment (start 112 132.25) (end 109.517677 129.767677) (width 1) (layer "B.Cu") (net 5))
   (segment (start 126 130.25) (end 129.25 127) (width 1) (layer "B.Cu") (net 5))
+  (segment (start 126.365 116.205) (end 126.365 120.65) (width 1) (layer "B.Cu") (net 5))
   (segment (start 104.81 92.69) (end 104.81 96.13) (width 1) (layer "B.Cu") (net 6))
   (segment (start 104.81 96.13) (end 107.37 98.69) (width 1) (layer "B.Cu") (net 6))
@@
   (segment (start 130.87 60.62) (end 130.87 67.25) (width 1) (layer "B.Cu") (net 23))
   (segment (start 128 59.25) (end 129.5 59.25) (width 1) (layer "B.Cu") (net 23))
+  (zone (net 1) (net_name "Earth") (layer "F.Cu") (hatch edge 0.508)
+    (connect_pads (clearance 0.508))
+    (min_thickness 0.254) (filled_areas_thickness no)
+    (fill yes (thermal_gap 0.508) (thermal_bridge_width 0.508))
+    (polygon
+      (pts
+        (xy 150.495 153.035)
+        (xy 99.06 153.035)
+        (xy 99.06 39.37)
+        (xy 150.495 39.37)
+      )
+    )
+  )
   (zone (net 1) (net_name "Earth") (layer "B.Cu") (hatch edge 0.508)
     (connect_pads (clearance 0.508))

Commit message: Ultra Fuzz and PTC files
Changed lines of the file:
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@@
     (fp_line (start -2.16 2.55) (end -2.16 4.05) (layer "F.Fab") (width 0.1))
     (fp_line (start -2.42 1.79) (end -2.42 2.55) (layer "F.Fab") (width 0.1))
-    (pad "1" thru_hole roundrect (at 0 0) (size 1.74 1.74) (drill 1.09) (layers *.Cu *.Mask) (roundrect_rratio 0.143678)
+    (pad "1" thru_hole roundrect (at 0 0) (size 1.74 1.74) (drill 1.09) (layers *.Cu *.Mask) (roundrect_rratio 0.1436781609)
       (net 8 "Net-(J2-Pad1)") (pinfunction "Pin_1") (pintype "passive"))
     (pad "2" thru_hole circle (at 2.54 0) (size 1.74 1.74) (drill 1.09) (layers *.Cu *.Mask)
@@
     (fp_line (start -2.29 -0.24) (end -2.29 1.79) (layer "F.Fab") (width 0.1))
     (fp_line (start 4.96 -2.55) (end -2.42 -2.55) (layer "F.Fab") (width 0.1))
-    (pad "1" thru_hole roundrect (at 0 0) (size 1.74 1.74) (drill 1.09) (layers *.Cu *.Mask) (roundrect_rratio 0.143678)
+    (pad "1" thru_hole roundrect (at 0 0) (size 1.74 1.74) (drill 1.09) (layers *.Cu *.Mask) (roundrect_rratio 0.1436781609)
       (net 21 "Net-(R3-Pad2)") (pinfunction "Pin_1") (pintype "passive"))
     (pad "2" thru_hole circle (at 2.54 0) (size 1.74 1.74) (drill 1.09) (layers *.Cu *.Mask)
@@
     (fp_line (start 4.83 -0.24) (end 4.96 -0.24) (layer "F.Fab") (width 0.1))
     (fp_line (start 0.5 -2.55) (end 0 -1.842893) (layer "F.Fab") (width 0.1))
-    (pad "1" thru_hole roundrect (at 0 0) (size 1.74 1.74) (drill 1.09) (layers *.Cu *.Mask) (roundrect_rratio 0.143678)
+    (pad "1" thru_hole roundrect (at 0 0) (size 1.74 1.74) (drill 1.09) (layers *.Cu *.Mask) (roundrect_rratio 0.1436781609)
       (net 21 "Net-(R3-Pad2)") (pinfunction "Pin_1") (pintype "passive"))
     (pad "2" thru_hole circle (at 2.54 0) (size 1.74 1.74) (drill 1.09) (layers *.Cu *.Mask)
@@
     (fp_line (start 7.45 -0.24) (end 7.58 -0.24) (layer "F.Fab") (width 0.1))
     (fp_line (start 7.58 2.55) (end 7.58 1.79) (layer "F.Fab") (width 0.1))
-    (pad "1" thru_hole roundrect (at 0 0) (size 1.74 1.74) (drill 1.09) (layers *.Cu *.Mask) (roundrect_rratio 0.143678)
+    (pad "1" thru_hole roundrect (at 0 0) (size 1.74 1.74) (drill 1.09) (layers *.Cu *.Mask) (roundrect_rratio 0.1436781609)
       (net 9 "Net-(R2-Pad2)") (pinfunction "Pin_1") (pintype "passive"))
     (pad "2" thru_hole circle (at 2.54 0) (size 1.74 1.74) (drill 1.09) (layers *.Cu *.Mask)
@@
     (fp_line (start -2.16 4.05) (end 4.7 4.05) (layer "F.Fab") (width 0.1))
     (fp_line (start -2.29 -0.24) (end -2.29 1.79) (layer "F.Fab") (width 0.1))
-    (pad "1" thru_hole roundrect (at 0 0) (size 1.74 1.74) (drill 1.09) (layers *.Cu *.Mask) (roundrect_rratio 0.143678)
+    (pad "1" thru_hole roundrect (at 0 0) (size 1.74 1.74) (drill 1.09) (layers *.Cu *.Mask) (roundrect_rratio 0.1436781609)
       (net 5 "+VDC") (pinfunction "Pin_1") (pintype "passive"))
     (pad "2" thru_hole circle (at 2.54 0) (size 1.74 1.74) (drill 1.09) (layers *.Cu *.Mask)
@@
     (fp_line (start -2.42 -2.55) (end -2.42 -0.24) (layer "F.Fab") (width 0.1))
     (fp_line (start 4.96 -2.55) (end -2.42 -2.55) (layer "F.Fab") (width 0.1))
-    (pad "1" thru_hole roundrect (at 0 0) (size 1.74 1.74) (drill 1.09) (layers *.Cu *.Mask) (roundrect_rratio 0.143678)
+    (pad "1" thru_hole roundrect (at 0 0) (size 1.74 1.74) (drill 1.09) (layers *.Cu *.Mask) (roundrect_rratio 0.1436781609)
       (net 6 "Net-(J1-Pad1)") (pinfunction "Pin_1") (pintype "passive"))
     (pad "2" thru_hole circle (at 2.54 0) (size 1.74 1.74) (drill 1.09) (layers *.Cu *.Mask)
