File: PASS_TONE_CTRL/Hardware/PASS_TONE_CTRL/PASS_TONE_CTRL.kicad_pcb (KiCad board)
At the start: 2 copper layers, 50 x 112 mm, 20 parts, among them J1 Input, J2 FREQ_A, J3 FREQ_B, J4 FREQ_COMM, J5 COIL_SW, J6 Output

Commit message: Ultra Fuzz and PTC files
Parts:
- added C1: 4.7nF, Capacitor_THT:C_Disc_D5.0mm_W2.5mm_P5.00mm, F.Cu at (106.0, 94.0)
- added C5: 68nF, Capacitor_THT:C_Disc_D5.0mm_W2.5mm_P5.00mm, F.Cu at (121.4, 99.1)
- added C9: 680nF, Capacitor_THT:C_Disc_D5.0mm_W2.5mm_P5.00mm, F.Cu at (138.7, 99.1)
- AUDIO TRANSFORMER: renamed from TR1; footprint RF_Mini-Circuits:Mini-Circuits_CD637_H5.23mm -> PassiveTonalControl:AudioTransformer_Thru
- J2: footprint Connector_Molex:Molex_SL_171971-0003_1x03_P2.54mm_Vertical -> Connector_Molex:Molex_SL_171971-0004_1x04_P2.54mm_Vertical
- J4: footprint Connector_Molex:Molex_SL_171971-0002_1x02_P2.54mm_Vertical -> Connector_Molex:Molex_SL_171971-0003_1x03_P2.54mm_Vertical
- R6: value DEPTH -> DEPTH 50k
- moved J6 36.1 mm to (136.4, 119.2)
- moved R6 33.1 mm to (137.2, 75.2)
- moved J1 32.8 mm to (111.5, 119.5)
- moved R1 31.3 mm to (109.7, 112.4)
- moved C6 24.5 mm to (126.5, 99.1), turned to 90 degrees
- moved C4 24.5 mm to (117.3, 99.1), turned to 90 degrees
- moved J3 21.9 mm to (123.6, 86.2)
- moved J5 16.9 mm to (108.2, 75.2)
- moved J2 16.5 mm to (108.2, 86.2)
- moved AUDIO TRANSFORMER 14.5 mm to (126.0, 63.0), turned to 180 degrees
- moved C10 14.4 mm to (142.7, 99.1), turned to 90 degrees
- moved C3 13.6 mm to (113.5, 99.0), turned to 90 degrees
- moved J4 12.2 mm to (139.0, 86.5)
- moved C8 11.8 mm to (134.6, 99.1), turned to 90 degrees
- moved C7 8.14 mm to (130.6, 99.1), turned to 90 degrees
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- renumbered C7 to C10, C1 to C2, C2 to C3, C3 to C4, C4 to C6, C5 to C7, C6 to C8
Connections:
- C10 pad 2: Net-(C7-Pad2) -> Net-(C10-Pad2)
- C2 pad 1: Net-(C1-Pad1) -> Net-(C2-Pad1)
- C3 pad 2: Net-(C2-Pad2) -> Net-(C3-Pad2)
- C4 pad 2: Net-(C3-Pad2) -> Net-(C4-Pad2)
- C6 pad 2: Net-(C4-Pad2) -> Net-(C6-Pad2)
- C7 pad 2: Net-(C5-Pad2) -> Net-(C7-Pad2)
- C8 pad 2: Net-(C6-Pad2) -> Net-(C8-Pad2)
- J2 pad 2: Net-(C2-Pad2) -> Net-(C2-Pad1)
- J3 pad 1: Net-(C4-Pad2) -> Net-(C5-Pad2)
- J3 pad 2: Net-(C5-Pad2) -> Net-(C6-Pad2)
- J3 pad 3: Net-(C6-Pad2) -> Net-(C7-Pad2)
- J3 pad 4: Net-(C7-Pad2) -> Net-(C8-Pad2)
- J4 pad 1: Net-(J4-Pad1) -> Net-(C9-Pad2)
- J4 pad 2: unconnected-(J4-Pad2) -> Net-(C10-Pad2)
- J5 pad 2: Net-(J4-Pad1) -> Net-(J5-Pad2)
Routing:
- net Net-(C8-Pad1): track 0.00 -> 71.0 mm
- net Net-(J5-Pad2): track 0.00 -> 42.4 mm
- net Net-(J5-Pad1): track 0.00 -> 32.6 mm
- net Net-(R6-Pad3): track 0.00 -> 24.8 mm
- net Net-(J5-Pad3): track 0.00 -> 20.6 mm
- net Net-(C8-Pad2): track 0.00 -> 10.4 mm
- net Net-(C1-Pad1): track 0.00 -> 9.22 mm
- net Net-(C5-Pad2): track 0.00 -> 9.18 mm
- net Net-(C4-Pad2): track 0.00 -> 8.69 mm
- net Net-(C7-Pad2): track 0.00 -> 8.60 mm
- net Net-(C2-Pad1): track 0.00 -> 8.19 mm
- net Net-(C10-Pad2): track 0.00 -> 8.08 mm
- net Net-(C6-Pad2): track 0.00 -> 7.97 mm
- net Net-(C3-Pad2): track 0.00 -> 7.88 mm
- net Net-(J1-Pad1): track 0.00 -> 7.86 mm
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- added copper zone on F.Cu, net Earth
Other:
- board text added: "Ezer Longinus Feb 2023"
- board text removed: "Ezer Longinus Jan 2023"
