File: PASS_TONE_CTRL/Hardware/PASS_TONE_CTRL/PASS_TONE_CTRL.kicad_sch (KiCad schematic)
At the start: 20 parts, among them J1 Input, J2 FREQ_A, J3 FREQ_B, J4 FREQ_COMM, J5 COIL_SW, J6 Output

Commit message: Ultra Fuzz and PTC files
Parts:
- removed J2: FREQ_A, Connector_Molex:Molex_SL_171971-0003_1x03_P2.54mm_Vertical, symbol Connector:Conn_01x03_Male
- removed J4: FREQ_COMM, Connector_Molex:Molex_SL_171971-0002_1x02_P2.54mm_Vertical, symbol Connector:Conn_01x02_Male
- added C1: 4.7nF, Capacitor_THT:C_Disc_D5.0mm_W2.5mm_P5.00mm, symbol Device:C_Small
- added C5: 68nF, Capacitor_THT:C_Disc_D5.0mm_W2.5mm_P5.00mm, symbol Device:C_Small
- added C9: 680nF, Capacitor_THT:C_Disc_D5.0mm_W2.5mm_P5.00mm, symbol Device:C_Small
- added J2: FREQ_A, Connector_Molex:Molex_SL_171971-0004_1x04_P2.54mm_Vertical, symbol Connector:Conn_01x04_Male
- added J4: FREQ_COMM, Connector_Molex:Molex_SL_171971-0003_1x03_P2.54mm_Vertical, symbol Connector:Conn_01x03_Male
- R6: value DEPTH -> DEPTH 50k
- TR1: footprint RF_Mini-Circuits:Mini-Circuits_CD637_H5.23mm -> PassiveTonalControl:AudioTransformer_Thru
- renumbered C7 to C10, C1 to C2, C2 to C3, C3 to C4, C4 to C6, C5 to C7, C6 to C8
Connections:
- net at C2.1: now also J2.2 (Pin_2)
- net at C10.1, C2.2, C3.1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: now also C1.2, C5.1, C9.1
- net at C3.2: now also J2.3 (Pin_3)
- net at J3.1 (Pin_1): now also C5.2; no longer C6.2
- net at J3.2 (Pin_2): now also C6.2; no longer C7.2
- net at J3.3 (Pin_3): now also C7.2; no longer C8.2
- net at J3.4 (Pin_4): now also C8.2; no longer C10.2
- net at C4.2: now also J2.4 (Pin_4)
- net at J5.2 (Pin_2): now also J4.3 (Pin_3)
- new net: C1.1, J2.1 (Pin_1)
- new net: C9.2, J4.1 (Pin_1)
- new net: C10.2, J4.2 (Pin_2)
Other:
- moved on the sheet: C10, C2, C3, C4, C6, C7, C8, J3
