File: ULTRA_FUZZ/Hardware/ULTRA_FUZZ/ULTRA_FUZZ.kicad_pcb (KiCad board)
At the start: 2 copper layers, 50 x 112 mm, 45 parts, among them J1 Input, J2 Meter Input, J3 Conn_02x08_Odd_Even, J4 FX Input, J5 Meter Output, J6 Output, J7 BALANCED OUTPUT, J8 Power LED, U1 TL074

Commit message: Ultra Fuzz and PTC files
Parts:
- removed C11: 1uF, Capacitor_THT:C_Disc_D5.0mm_W2.5mm_P5.00mm
- removed C12, C7, C8: 10uF, Capacitor_THT:CP_Radial_D8.0mm_P3.80mm
- removed C4: 220nF, Capacitor_THT:C_Disc_D5.0mm_W2.5mm_P5.00mm
- removed C5: 2.2uF, Capacitor_THT:CP_Radial_D8.0mm_P3.80mm
- removed D5, D6: 1N4148, Diode_THT:D_DO-35_SOD27_P7.62mm_Horizontal
- removed J5: Meter Output, Connector_Molex:Molex_SL_171971-0002_1x02_P2.54mm_Vertical
- removed J6: Output, Connector_Molex:Molex_SL_171971-0002_1x02_P2.54mm_Vertical
- removed J7: BALANCED OUTPUT, Connector_Molex:Molex_SL_171971-0003_1x03_P2.54mm_Vertical
- removed JP1: Jumper_2_Open, Connector_PinSocket_2.54mm:PinSocket_1x02_P2.54mm_Vertical
- removed R12: 1M, Potentiometer_THT:Potentiometer_Piher_PT-10-V10_Vertical
- removed S1: CLEAN/DIRTY, Connector_Molex:Molex_SL_171971-0002_1x02_P2.54mm_Vertical
- added Q1: 2N5457, Package_TO_SOT_THT:TO-92L_Inline_Wide, F.Cu at (122.5, 63.5)
- added SW1A1: BYPASS_A, Connector_Molex:Molex_SL_171971-0003_1x03_P2.54mm_Vertical, F.Cu at (116.2, 76.0)
- added SW1B1: BYPASS_B, Connector_Molex:Molex_SL_171971-0003_1x03_P2.54mm_Vertical, F.Cu at (129.2, 76.0)
- C1: value 4.7pF -> 47pF
- C2: value 4.7pF -> 100nF
- C3: value 100nF -> 220nF
- D1, D2: value LED -> 1N914; footprint LED_THT:LED_D5.0mm -> Diode_THT:D_DO-35_SOD27_P7.62mm_Horizontal
- J1: value Input -> INPUT
- J2: value Meter Input -> OUTPUT
- J4: value FX Input -> BYPASS LED
- J8: value Power LED -> POWER LED
- R1: value 1k -> 10k
- R10: value 470k -> 22M
- R11: value 1M -> 2k2
- R2: value 4k7 -> 10k
- R4: footprint Resistor_THT:R_Axial_DIN0207_L6.3mm_D2.5mm_P7.62mm_Horizontal -> Connector_Molex:Molex_SL_171971-0003_1x03_P2.54mm_Vertical
- R5: value 1k -> 10k; footprint Resistor_THT:R_Axial_DIN0207_L6.3mm_D2.5mm_P7.62mm_Horizontal -> Connector_Molex:Molex_SL_171971-0003_1x03_P2.54mm_Vertical
- R6: value GAIN POT -> 100k; footprint Connector_Molex:Molex_SL_171971-0003_1x03_P2.54mm_Vertical -> Resistor_THT:R_Axial_DIN0207_L6.3mm_D2.5mm_P7.62mm_Horizontal
- R7: value MASTER -> 100k; footprint Connector_Molex:Molex_SL_171971-0003_1x03_P2.54mm_Vertical -> Resistor_THT:R_Axial_DIN0207_L6.3mm_D2.5mm_P7.62mm_Horizontal
- R8: value 100k -> 1M
- R9: value 470k -> 1k
- U1: value TL074 -> TL072; footprint Package_DIP:DIP-14_W7.62mm_LongPads -> Package_DIP:DIP-8_W7.62mm_Socket_LongPads
- moved R7 49.0 mm to (135.5, 113.7), turned to -90 degrees
- moved R6 44.2 mm to (117.3, 108.0), turned to 180 degrees
- moved J4 43.2 mm to (141.5, 56.5)
- moved J1 41.3 mm to (105.7, 76.0)
- moved C3 39.2 mm to (145.5, 115.0), turned to -90 degrees
- moved D2 37.8 mm to (121.2, 55.0)
- moved R8 37.6 mm to (120.7, 131.0), turned to 0 degrees
- moved R5 37.5 mm to (139.5, 90.0), turned to 0 degrees
- moved J2 36.7 mm to (142.2, 76.0)
- moved U1 34.0 mm to (128.8, 121.3), turned to 180 degrees
- moved R1 33.1 mm to (116.0, 121.3), turned to 90 degrees
- moved R10 29.4 mm to (129.3, 68.0), turned to 180 degrees
- moved D1 26.0 mm to (128.8, 58.5)
- moved R3 25.7 mm to (112.5, 104.0), turned to 90 degrees
- moved C1 23.5 mm to (127.0, 127.0)
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Connections:
- C1 pad 1: Earth -> Net-(R8-Pad2)
- C1 pad 2: Net-(C1-Pad2) -> Net-(R8-Pad1)
- C10 pad 2: Net-(C10-Pad2) -> VSS
- C2 pad 2: Net-(C2-Pad2) -> Net-(R8-Pad2)
- C3 pad 2: Net-(C1-Pad2) -> Net-(R7-Pad1)
- C6 pad 1: Net-(C2-Pad1) -> Net-(C6-Pad1)
- C9 pad 1: Net-(C9-Pad1) -> VDD
- D1 pad 2: Net-(C2-Pad2) -> Net-(D1-Pad2)
- D2 pad 1: Net-(C2-Pad2) -> Net-(D2-Pad1)
- D3 pad 1: Net-(C9-Pad1) -> VDD
- D4 pad 2: Net-(C10-Pad2) -> VSS
- J1 pad 1: Net-(C3-Pad1) -> Net-(J1-Pad1)
- J2 pad 1: Net-(C4-Pad2) -> Net-(SW1A1-Pad3)
- J4 pad 1: Earth -> Net-(J4-Pad1)
- J4 pad 2: Net-(J4-Pad2) -> Earth
- J8 pad 1: Net-(C9-Pad1) -> VDD
- R1 pad 1: Net-(J4-Pad2) -> Net-(C2-Pad1)
- R1 pad 2: Net-(C5-Pad1) -> Net-(R1-Pad2)
- R10 pad 1: Net-(C2-Pad2) -> Net-(SW1B1-Pad3)
- R10 pad 2: Net-(C2-Pad1) -> VDD
- R11 pad 1: Net-(C4-Pad2) -> Net-(J4-Pad1)
- R11 pad 2: Earth -> Net-(D2-Pad1)
- R2 pad 1: Net-(R2-Pad1) -> Net-(R4-Pad1)
- R2 pad 2: Net-(C2-Pad2) -> VSS
- R3 pad 1: Net-(R3-Pad1) -> VDD
- R3 pad 2: Net-(J6-Pad1) -> Net-(R4-Pad3)
- R4 pad 1: Net-(R3-Pad1) -> Net-(R4-Pad1)
- R4 pad 2: Net-(C7-Pad1) -> Net-(R4-Pad2)
- R5 pad 2: Net-(J8-Pad2) -> Net-(R5-Pad2)
- R6 pad 1: Earth -> Net-(R1-Pad2)
- R6 pad 2: Net-(R2-Pad1) -> Earth
- R7 pad 1: Earth -> Net-(R7-Pad1)
- R7 pad 2: Net-(J6-Pad1) -> Net-(R8-Pad1)
- R8 pad 1: Net-(C4-Pad1) -> Net-(R8-Pad1)
- R8 pad 2: Earth -> Net-(R8-Pad2)
- R9 pad 1: Net-(C1-Pad2) -> Earth
- R9 pad 2: Earth -> Net-(J8-Pad2)
- U1 pad 1: Net-(C5-Pad1) -> Net-(R8-Pad2)
- U1 pad 2: Net-(C5-Pad1) -> Net-(R8-Pad1)
- U1 pad 3: Net-(C1-Pad2) -> Earth
- U1 pad 4: Net-(C9-Pad1) -> VSS
- U1 pad 5: Net-(C4-Pad1) -> Net-(R1-Pad2)
- U1 pad 6: Net-(C8-Pad1) -> Net-(R4-Pad2)
- U1 pad 7: Net-(C8-Pad1) -> Net-(C6-Pad1)
- U1 pad 8: Net-(C2-Pad1) -> VDD
Routing:
- net Net-(J6-Pad1): track 159.9 -> 0.00 mm, vias 2 -> 0
- net VDD: track 0.00 -> 142.4 mm
- net Net-(C9-Pad1): track 131.7 -> 0.00 mm
- net VSS: track 0.00 -> 126.8 mm
- net Net-(C4-Pad2): track 92.6 -> 0.00 mm
- net Net-(C10-Pad2): track 88.4 -> 0.00 mm
- net Net-(C1-Pad2): track 80.5 -> 0.00 mm
- net Net-(C2-Pad2): track 75.1 -> 0.00 mm, vias 4 -> 0
- net Net-(C2-Pad1): track 77.2 -> 5.54 mm, vias 2 -> 0
- net Net-(J5-Pad1): track 71.1 -> 0.00 mm
- net Net-(C8-Pad2): track 60.5 -> 0.00 mm
- net Net-(C3-Pad1): track 6.76 -> 61.1 mm, vias 0 -> 2
- net Net-(R8-Pad2): track 0.00 -> 50.2 mm, vias 0 -> 2
- net Net-(C7-Pad1): track 42.8 -> 0.00 mm, vias 2 -> 0
- net Net-(SW1A1-Pad3): track 0.00 -> 39.3 mm, vias 0 -> 2
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Other:
- board text added: "EZER LONGINUS FEB 2023"
- board text added: "ULTRA FUZZ"
- board text removed: "EPFM - PREAMP"
- board text removed: "Ezer Longinus Feb 2023"
