File: ULTRA_FUZZ/Hardware/ULTRA_FUZZ/ULTRA_FUZZ.kicad_sch (KiCad schematic)
At the start: 45 parts, among them J1 Input, J2 Meter Input, J3 Conn_02x08_Odd_Even, J4 FX Input, J5 Meter Output, J6 Output, J7 BALANCED OUTPUT, J8 Power LED, U1 TL074

Commit message: Ultra Fuzz and PTC files
Parts:
- removed C11: 1uF, Capacitor_THT:C_Disc_D5.0mm_W2.5mm_P5.00mm, symbol Device:C_Small
- removed C12, C7, C8: 10uF, Capacitor_THT:CP_Radial_D8.0mm_P3.80mm, symbol Device:C_Polarized_Small_US
- removed C4: 220nF, Capacitor_THT:C_Disc_D5.0mm_W2.5mm_P5.00mm, symbol Device:C_Small
- removed C5: 2.2uF, Capacitor_THT:CP_Radial_D8.0mm_P3.80mm, symbol Device:C_Polarized_Small_US
- removed D1, D2: LED, LED_THT:LED_D5.0mm, symbol Device:LED
- removed D5, D6: 1N4148, Diode_THT:D_DO-35_SOD27_P7.62mm_Horizontal, symbol Diode:1N4148
- removed J2: Meter Input, Connector_Molex:Molex_SL_171971-0002_1x02_P2.54mm_Vertical, symbol Connector:Conn_01x02_Male
- removed J5: Meter Output, Connector_Molex:Molex_SL_171971-0002_1x02_P2.54mm_Vertical, symbol Connector:Conn_01x02_Male
- removed J7: BALANCED OUTPUT, Connector_Molex:Molex_SL_171971-0003_1x03_P2.54mm_Vertical, symbol Connector:Conn_01x03_Male
- removed JP1: Jumper_2_Open, Connector_PinSocket_2.54mm:PinSocket_1x02_P2.54mm_Vertical, symbol Jumper:Jumper_2_Open
- removed R12: 1M, Potentiometer_THT:Potentiometer_Piher_PT-10-V10_Vertical, symbol Device:R_Potentiometer_US
- removed R4: 10k, Resistor_THT:R_Axial_DIN0207_L6.3mm_D2.5mm_P7.62mm_Horizontal, symbol Device:R_Small_US
- removed S1: CLEAN/DIRTY, Connector_Molex:Molex_SL_171971-0002_1x02_P2.54mm_Vertical, symbol Connector:Conn_01x02_Male
- removed U1: TL074, Package_DIP:DIP-14_W7.62mm_LongPads, symbol Amplifier_Operational:TL074
- added D1, D2: 1N914, Diode_THT:D_DO-35_SOD27_P7.62mm_Horizontal, symbol Diode:1N914
- added Q1: 2N5457, Package_TO_SOT_THT:TO-92L_Inline_Wide, symbol Device:Q_NJFET_DSG
- added R10: 22M, Resistor_THT:R_Axial_DIN0207_L6.3mm_D2.5mm_P7.62mm_Horizontal, symbol Device:R_Small_US
- added SW1A1: BYPASS_A, Connector_Molex:Molex_SL_171971-0003_1x03_P2.54mm_Vertical, symbol Connector:Conn_01x03_Male
- added SW1B1: BYPASS_B, Connector_Molex:Molex_SL_171971-0003_1x03_P2.54mm_Vertical, symbol Connector:Conn_01x03_Male
- added U1: TL072, Package_DIP:DIP-8_W7.62mm_Socket_LongPads, symbol Amplifier_Operational:TL072
- C1: value 4.7pF -> 47pF
- C2: value 4.7pF -> 100nF
- C3: value 100nF -> 220nF
- J4: value FX Input -> Bypass LED
- R1: value 1k -> 10k
- R11: value 1M -> 2k2
- R2: value 4k7 -> 10k
- R4: renamed from R7; value MASTER -> 10k
- R5: renamed from R6; value GAIN POT -> 10k
- R6: renamed from R9; value 470k -> 100k
- R7: renamed from R10; value 470k -> 100k
- R8: value 100k -> 1M
- renumbered J6 to J2, R5 to R9
Connections:
- net Earth: now also J4.2 (Pin_2), U1.3 (+); no longer C1.1, J4.1 (Pin_1), R11.2, R4.1 (Pin_1), R8.2
- net at C3.1: now also SW1A1.1 (Pin_1); no longer J1.1 (Pin_1)
- net at R1.2: now also R6.1, U1.5 (+)
- net at R5.3 (Pin_3): now also C6.2
- net at R1.1: now also C2.1; no longer J4.2 (Pin_2)
- net at R8.1: now also C1.2, R7.2, U1.2 (-)
- net VDD: now reaches R3.1
- net VDD: now also C9.1, D3.1 (K), J8.1 (Pin_1), Q1.1 (D), R10.2, U1.8 (V+)
- net VSS: now reaches C10.2, D4.2 (A)
- net VSS: now also R2.2, U1.4 (V-)
- net at R4.3 (Pin_3): now also R3.2; no longer C6.2
- net at R11.1: now also J4.1 (Pin_1)
- net at R5.2 (Pin_2): now also SW1B1.2 (Pin_2); no longer R2.1
- new net: C3.2, R7.1
- new net: D2.1 (K), R11.2
- new net: D1.2 (A), Q1.2 (S)
- new net: Q1.3 (G), R10.1, SW1B1.3 (Pin_3)
- new net: C1.1, C2.2, R8.2, U1.1
- new net: C6.1, U1.7
- new net: J1.1 (Pin_1), SW1A1.2 (Pin_2)
- new net: R4.2 (Pin_2), U1.6 (-)
- new net: J2.1 (Pin_1), SW1A1.3 (Pin_3), SW1B1.1 (Pin_1)
- new net: R2.1, R4.1 (Pin_1)
- new net: D1.1 (K), D2.2 (A)
Other:
- note added: "OUTPUT"
- note added: "SENSITIVITY"
- note added: "ULTRA FUZZ"
- note removed: "PREAMP"
- moved on the sheet: C1, C2, C3, C6, H1, H2, H3, H4, J1, J2, R1, R2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
